File: PCB/Frogboard.kicad_pcb (KiCad board)
At the start: 2 copper layers, 323.9 x 133.4 mm, 353 parts, among them J1 SW_Push, K1 SW_Push, M1 SW_Push, P1 SW_Push, Q1 SW_Push, Q2 NMOS, SW0 SW_Push, SW1 SW_Push, SW10 RotaryEncoder_Switch_MP, SW11 SW_Push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

Commit message: Update PCB
Parts:
- moved A3 1.29 mm to (345.9, 70.1), turned to 90 degrees
Routing:
- net ROW0: track 309.7 -> 259.3 mm, vias 1 -> 2
- net ROW1: track 321.9 -> 272.8 mm
- net ROW3: track 328.3 -> 364.0 mm, vias 4 -> 1
- net 1B: track 22.0 -> 57.3 mm, vias 0 -> 3
- net +5V: track 2114.5 -> 2079.3 mm, vias 151 -> 148
- net 1A: track 22.8 -> 54.2 mm, vias 1 -> 2
- net NMOS_GATE: track 32.8 -> 7.94 mm, vias 1 -> 0
- net ROW4: track 334.5 -> 355.1 mm, vias 2 -> 4
- net LCD_DC: track 25.5 -> 41.1 mm
- net GND: track 2792.0 -> 2807.1 mm, vias 17 -> 15
- net 1S1: track 1911.8 -> 1897.8 mm, vias 26 -> 23
- net LED DIN: track 278.4 -> 292.0 mm
- net LCD_CLK: track 19.3 -> 30.2 mm, vias 0 -> 2
- net LCD_MOSI: track 16.1 -> 25.6 mm, vias 0 -> 2
- net Net-(USB1-CC2): track 32.4 -> 24.7 mm, vias 0 -> 2
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
Commit message: Update pcb
Parts:
- moved TP1 4.73 mm to (341.9, 58.2)
- moved TP2 4.23 mm to (341.9, 54.0)
Routing:
- net D-: track 19.7 -> 14.2 mm, vias 1 -> 0
- net D+: track 12.9 -> 12.1 mm
Changed lines of the file:
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@@
 	(footprint "TestPoint:TestPoint_Pad_D2.0mm"
 		(layer "F.Cu")
-		(at 341.906207 53.470223)
+		(at 341.906207 58.2)
 		(descr "SMD pad as test Point, diameter 2.0mm")
 		(tags "test point SMD pad")
@@
 	(footprint "TestPoint:TestPoint_Pad_D2.0mm"
 		(layer "F.Cu")
-		(at 341.906207 58.232723)
+		(at 341.906207 54)
 		(descr "SMD pad as test Point, diameter 2.0mm")
 		(tags "test point SMD pad")
@@
 	)
 	(segment
-		(start 351.011207 57.329354)
-		(end 351.011207 57.788973)
+		(start 350.420826 56.738973)
+		(end 351.011207 57.329354)
 		(width 0.2)
 		(layer "F.Cu")
@@
 	)
 	(segment
-		(start 349.880826 56.198973)
-		(end 351.011207 57.329354)
+		(start 341.906207 58.2)
+		(end 343.367234 56.738973)
 		(width 0.2)
 		(layer "F.Cu")
@@
 	)
 	(segment
-		(start 351.011207 57.788973)
-		(end 351.011207 58.255089)
+		(start 351.851207 59.095089)
+		(end 351.851207 59.138973)
 		(width 0.2)
 		(layer "F.Cu")
@@
 	)
 	(segment
-		(start 341.906207 53.470223)
-		(end 344.634957 56.198973)
+		(start 351.011207 58.255089)
+		(end 351.851207 59.095089)
 		(width 0.2)
 		(layer "F.Cu")
@@
 	)
 	(segment
-		(start 344.634957 56.198973)
-		(end 349.880826 56.198973)
+		(start 351.011207 57.329354)
+		(end 351.011207 57.788973)
 		(width 0.2)
 		(layer "F.Cu")
@@
 	)
 	(segment
-		(start 351.011207 58.255089)
-		(end 351.851207 59.095089)
+		(start 351.011207 57.788973)
+		(end 351.011207 58.255089)
 		(width 0.2)
 		(layer "F.Cu")
@@
 	)
 	(segment
-		(start 351.851207 59.095089)
-		(end 351.851207 59.138973)
+		(start 343.367234 56.738973)
+		(end 350.420826 56.738973)
 		(width 0.2)
 		(layer "F.Cu")
@@
 	)
 	(segment
-		(start 344.232723 58.232723)
-		(end 344.5 58.5)
+		(start 341.906207 54)
+		(end 344.10518 56.198973)
 		(width 0.2)
 		(layer "F.Cu")
@@
 	)
 	(segment
-		(start 341.906207 58.232723)
-		(end 344.232723 58.232723)
+		(start 351.851207 57.603668)
+		(end 351.851207 57.788973)
 		(width 0.2)
 		(layer "F.Cu")
 		(net "D-")
 	)
-	(via
-		(at 344.5 58.5)
-		(size 0.6)
-		(drill 0.3)
-		(layers "F.Cu" "B.Cu")
+	(segment
+		(start 350.446512 56.198973)
+		(end 351.851207 57.603668)
+		(width 0.2)
+		(layer "F.Cu")
 		(net "D-")
 	)
 	(segment
-		(start 351.851207 57.832857)
-		(end 351.851207 57.788973)
+		(start 344.10518 56.198973)
+		(end 350.446512 56.198973)
 		(width 0.2)
-		(layer "B.Cu")
+		(layer "F.Cu")
 		(net "D-")
 	)
 	(segment
-		(start 347.50471 52.798973)
-		(end 351.636207 56.93047)
+		(start 351.851207 57.832857)
+		(end 351.851207 57.788973)
 		(width 0.2)
 		(layer "B.Cu")
@@
 	)
 	(segment
-		(start 344.5 55.016677)
-		(end 346.717704 52.798973)
-		(width 0.2)
-		(layer "B.Cu")
-		(net "D-")
-	)
-	(segment
 		(start 351.011207 58.672857)
 		(end 351.011207 59.138973)
 		(width 0.2)
 		(layer "B.Cu")
-		(net "D-")
-	)
-	(segment
-		(start 351.636207 56.93047)
-		(end 351.636207 58.047857)
-		(width 0.2)
-		(layer "B.Cu")
-		(net "D-")
-	)
-	(segment
-		(start 344.5 58.5)
-		(end 344.5 55.016677)
-		(width 0.2)
-		(layer "B.Cu")
-		(net "D-")
-	)
-	(segment
-		(start 346.717704 52.798973)
-		(end 347.50471 52.798973)
-		(width 0.2)
-		(layer "B.Cu")

Commit message: update pcb
Routing:
- net Net-(USB1-CC2): track 24.7 -> 23.9 mm
Changed lines of the file:
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@@
 	)
 	(setup
+		(stackup
+			(layer "F.SilkS"
+				(type "Top Silk Screen")
+			)
+			(layer "F.Paste"
+				(type "Top Solder Paste")
+			)
+			(layer "F.Mask"
+				(type "Top Solder Mask")
+				(thickness 0.01)
+			)
+			(layer "F.Cu"
+				(type "copper")
+				(thickness 0.035)
+			)
+			(layer "dielectric 1"
+				(type "core")
+				(thickness 1.51)
+				(material "FR4")
+				(epsilon_r 4.5)
+				(loss_tangent 0.02)
+			)
+			(layer "B.Cu"
+				(type "copper")
+				(thickness 0.035)
+			)
+			(layer "B.Mask"
+				(type "Bottom Solder Mask")
+				(thickness 0.01)
+			)
+			(layer "B.Paste"
+				(type "Bottom Solder Paste")
+			)
+			(layer "B.SilkS"
+				(type "Bottom Silk Screen")
+			)
+			(copper_finish "None")
+			(dielectric_constraints no)
+		)
 		(pad_to_mask_clearance 0)
 		(allow_soldermask_bridges_in_footprints no)
@@
 		(capping no)
 		(filling no)
+		(zone_defaults)
 		(pcbplotparams
 			(layerselection 0x00000000_00000000_55555555_5755f5ff)
@@
 	)
 	(segment
-		(start 350.420826 56.738973)
-		(end 351.011207 57.329354)
+		(start 351.011207 57.58537)
+		(end 351.011207 57.788973)
 		(width 0.2)
 		(layer "F.Cu")
@@
 	)
 	(segment
-		(start 341.906207 58.2)
-		(end 343.367234 56.738973)
+		(start 351.011207 58.298973)
+		(end 351.851207 59.138973)
 		(width 0.2)
 		(layer "F.Cu")
@@
 	)
 	(segment
-		(start 351.011207 58.255089)
-		(end 351.851207 59.095089)
+		(start 346.531316 56.648953)
+		(end 350.07479 56.648953)
 		(width 0.2)
 		(layer "F.Cu")
@@
 	)
 	(segment
-		(start 351.011207 57.329354)
-		(end 351.011207 57.788973)
+		(start 341.906207 58.2)
+		(end 343.781206 56.325001)
 		(width 0.2)
 		(layer "F.Cu")
@@
 	)
 	(segment
-		(start 351.011207 57.788973)
-		(end 351.011207 58.255089)
+		(start 343.781206 56.325001)
+		(end 346.207364 56.325001)
+		(width 0.2)
+		(layer "F.Cu")
+		(net "D+")
+	)
+	(segment
+		(start 346.207364 56.325001)
+		(end 346.531316 56.648953)
+		(width 0.2)
+		(layer "F.Cu")
+		(net "D+")
+	)
+	(segment
+		(start 350.07479 56.648953)
+		(end 351.011207 57.58537)
 		(width 0.2)
 		(layer "F.Cu")
@@
 	)
 	(segment
-		(start 343.367234 56.738973)
-		(end 350.420826 56.738973)
+		(start 351.011207 57.788973)
+		(end 351.011207 58.298973)
 		(width 0.2)
 		(layer "F.Cu")
@@
 	)
 	(segment
-		(start 341.906207 54)
-		(end 344.10518 56.198973)
+		(start 349.613259 56.198973)
+		(end 349.937233 55.874999)
+		(width 0.2)
+		(layer "F.Cu")
+		(net "D-")
+	)
+	(segment
+		(start 346.717704 56.198973)
+		(end 349.613259 56.198973)
+		(width 0.2)
+		(layer "F.Cu")
+		(net "D-")
+	)
+	(segment
+		(start 343.781206 55.874999)
+		(end 346.39373 55.874999)
 		(width 0.2)
 		(layer "F.Cu")
@@
 	)
 	(segment
-		(start 350.446512 56.198973)
-		(end 351.851207 57.603668)
+		(start 346.39373 55.874999)
+		(end 346.717704 56.198973)
 		(width 0.2)
 		(layer "F.Cu")
@@
 	)
 	(segment
-		(start 344.10518 56.198973)
-		(end 350.446512 56.198973)
+		(start 341.906207 54)
+		(end 343.781206 55.874999)
+		(width 0.2)
+		(layer "F.Cu")
+		(net "D-")
+	)
+	(segment
+		(start 349.937233 55.874999)
+		(end 351.851207 57.788973)
 		(width 0.2)
 		(layer "F.Cu")
@@
 	(segment
 		(start 350 54.5)
-		(end 349 55.5)
+		(end 351 54.5)
 		(width 0.2)
 		(layer "F.Cu")
@@
 	)
 	(segment
-		(start 351 54.5)
+		(start 349.75 54.75)
 		(end 350 54.5)
 		(width 0.2)
@@
 	)
 	(via
-		(at 349 55.5)
+		(at 349.75 54.75)
 		(size 0.6)
 		(drill 0.3)
@@
 	)
 	(segment
-		(start 356.14471 60.538973)
-		(end 356.701207 59.982476)
+		(start 350.151207 56.651207)
+		(end 350.151207 57.788973)
 		(width 0.2)
 		(layer "B.Cu")
@@
 	)
 	(segment
-		(start 356.14471 63.640726)
-		(end 356.14471 60.538973)
+		(start 356.14471 60.538973)
+		(end 356.701207 59.982476)
 		(width 0.2)
 		(layer "B.Cu")
@@
 	)
 	(segment
-		(start 350.151207 56.651207)
-		(end 350.151207 57.788973)
+		(start 356.14471 63.640726)
+		(end 356.14471 60.538973)
 		(width 0.2)
 		(layer "B.Cu")
@@
 	)
 	(segment
-		(start 349 55.5)
-		(end 350.151207 56.651207)
-		(width 0.2)
-		(layer "B.Cu")
-		(net "Net-(USB1-CC2)")
-	)
-	(segment
 		(start 356.701207 59.982476)
 		(end 356.701207 57.29547)
@@
 		(width 0.2)
 		(layer "B.Cu")
+		(net "Net-(USB1-CC2)")
+	)
+	(segment
+		(start 349.75 54.75)
+		(end 350.151207 56.651207)
+		(width 0.2)
+		(layer "B.Cu")
